File: kicad/monitor-esp32/monitor.kicad_pcb (KiCad board)
At the start: 2 copper layers, 19.5 x 37.7 mm, 24 parts, among them J1 Conn, J2 Conn_01x14, J5 Conn, Q1 Q_NPN_BEC, Q2 IRLML0060TRPBF, T1 B82801A150, U1 AD8541

Commit message: изменено:      kicad/monitor-esp32/monitor-cache.lib 	изменено:      kicad/monitor-esp32/monitor.kicad_pcb 	изменено:      kicad/monitor-esp32/monitor.kicad_pcb-bak 	изменено:      kicad/monitor-esp32/monitor.sch 	изменено:      kicad/monitor-esp32/monitor.sch-bak
Parts:
- C1: value 200 -> 100
- Q2: value IRLML0060TRPBF -> IRLML6346
- R4: footprint Resistor_SMD:R_2512_6332Metric -> Resistor_SMD:R_1206_3216Metric
- R6: value 10M -> 30M
- moved R4 0.53 mm to (36.0, 78.0)
Connections:
- net Net-(J2-Pad11) renamed /ESP32.port.27
Routing:
- net GND: track 70.0 -> 79.2 mm
- net Net-(C6-Pad1): track 6.92 -> 8.25 mm
- net Net-(C5-Pad1): track 5.15 -> 6.12 mm
