File: kicad/monitor-esp32/monitor.sch (KiCad schematic (older format))
At the start: 24 parts, among them J1 Conn, J2 Conn_01x14, J5 Conn, Q1 Q_NPN_BEC, Q2 IRLML6346, T1 B82801A150, U1 AD8541

Commit message: изменено:      kicad/monitor-esp32/monitor-cache.lib 	изменено:      kicad/monitor-esp32/monitor.kicad_pcb 	изменено:      kicad/monitor-esp32/monitor.kicad_pcb-bak 	изменено:      kicad/monitor-esp32/monitor.sch 	изменено:      kicad/monitor-esp32/monitor.sch-bak
Parts:
- R4: value 5G -> RH73W2A5GNTN; footprint Resistor_SMD:R_2512_6332Metric -> Resistor_SMD:R_1206_3216Metric
Changed lines of the file:
@@
 U 1 1 60E0BE31
 P 7600 2000
-F 0 "R4" V 7393 2000 50  0000 C CNN
-F 1 "5G" V 7484 2000 50  0000 C CNN
-F 2 "Resistor_SMD:R_2512_6332Metric" V 7530 2000 50  0001 C CNN
+F 0 "R4" V 7500 2000 50  0000 C CNN
+F 1 "RH73W2A5GNTN" V 7700 1800 50  0000 C CNN
+F 2 "Resistor_SMD:R_1206_3216Metric" V 7530 2000 50  0001 C CNN
 F 3 "~" H 7600 2000 50  0001 C CNN
 	1    7600 2000

Commit message: изменено:      kicad/monitor-esp32/monitor.sch 	изменено:      kicad/monitor-esp32/monitor.sch-bak
Parts:
- R4: value RH73W2A5GNTN -> HVC1206Z5007KET
Changed lines of the file:
@@
 P 7600 2000
 F 0 "R4" V 7500 2000 50  0000 C CNN
-F 1 "RH73W2A5GNTN" V 7700 1800 50  0000 C CNN
+F 1 "HVC1206Z5007KET" V 7700 1750 50  0000 C CNN
 F 2 "Resistor_SMD:R_1206_3216Metric" V 7530 2000 50  0001 C CNN
 F 3 "~" H 7600 2000 50  0001 C CNN
